Commit message: added gazebo_control

File: src/my_robot/description/robot.urdf.xacro (robot description, xacro)
@@ -2,3 +2,4 @@
 <robot xmlns:xacro="http://www.ros.org/wiki/xacro" name ="robot">
    <xacro:include filename="robot_core.xacro" />
+   <xacro:include filename="gazebo_control.xacro" />
 </robot>

File: src/my_robot/description/robot_core.xacro (robot description, xacro)
@@ -280,12 +280,12 @@
         rpy="0 0 0" />
       <mass
-        value="0" />
-      <inertia
-        ixx="0"
-        ixy="0"
-        ixz="0"
-        iyy="0"
+        value="0.5" />
+      <inertia
+        ixx="0.0"
+        ixy="0.0"
+        ixz="0.0"
+        iyy="0.0"
         iyz="0"
-        izz="0" />
+        izz="0.0" />
     </inertial>
     <visual>
@@ -314,5 +314,5 @@
   <joint
     name="turr_joint"
-    type="revolute">
+    type="fixed">
     <origin
       xyz="0.23735 -0.74397 0.30328"
