Commit message: modified urdf and added lidar(only lidar)

File: src/my_robot/description/gazebo_control.xacro (robot description, xacro)
@@ -2,13 +2,18 @@
 <robot xmlns:xacro="http://www.ros.org/wiki/xacro" >
 	<gazebo>
-		<plugin name="my_robot" filename="libgazebo_ros_diff_drive.so" >
-            <left_joint>w_joint_1</left_joint>
-            <left_joint>w_joint_3</left_joint>
-            <right_joint>w_joint_2</right_joint>
-            <right_joint>w_joint_4</right_joint>
-            <wheel_separation>0.82</wheel_separation>
-            <wheel_diamenter>0.1</wheel_diamenter>
-            <max_wheel_torque>200<max_wheel_torque>
-            <max_wheel_acceleration>10.0<max_wheel_acceleration>
+		<plugin name="diff_drive" filename="libgazebo_ros_diff_drive.so" >
+            <ros>
+                  <namespace>/</namespace>
+                  <remapping>cmd_vel:=/cmd_vel</remapping>
+            </ros>
+            <num_wheel_pairs>2</num_wheel_pairs>
+            <left_joint>JOINT_WHEEL_1</left_joint>
+            <left_joint>JOINT_WHEEL_3</left_joint>
+            <right_joint>JOINT_WHEEL_2</right_joint>
+            <right_joint>JOINT_WHEEL_4</right_joint>
+            <wheel_separation>0.60</wheel_separation>
+            <wheel_diameter>0.1</wheel_diameter>
+            <max_wheel_torque>200</max_wheel_torque>
+            <max_wheel_acceleration>10.0</max_wheel_acceleration>
             <odometry_frame>odom</odometry_frame>
             <robot_base_frame>base_link</robot_base_frame>
@@ -17,4 +22,9 @@
             <publish_wheel_tf>true</publish_wheel_tf>
 		</plugin>
+            <plugin name="move_target" filename="libgazebo_ros_force_system.so">
+                  <body_name>TURRET</body_name>
+                  <reference_frame>world</reference_frame>
+                  <force>0 5 0</force>
+            </plugin>
 	</gazebo>
 </robot>

File: src/my_robot/description/robot.urdf.xacro (robot description, xacro)
@@ -3,3 +3,4 @@
    <xacro:include filename="robot_core.xacro" />
    <xacro:include filename="gazebo_control.xacro" />
+   <xacro:include filename="lidar.xacro"/>
 </robot>

File: src/my_robot/description/robot_core.xacro (robot description, xacro)
@@ -1,19 +1,23 @@
-<?xml version="1.0"?>
-<robot xmlns:xacro="http://www.ros.org/wiki/xacro">
+<?xml version="1.0" encoding="utf-8"?>
+<!-- This URDF was automatically created by SolidWorks to URDF Exporter! Originally created by Stephen Brawner (brawner@gmail.com)
+     Commit Version: 1.6.0-4-g7f85cfe  Build Version: 1.6.7995.38578
+     For more information, please see http://wiki.ros.org/sw_urdf_exporter -->
+<robot
+  name="ieee">
   <link
     name="base_link">
     <inertial>
       <origin
-        xyz="0.23811 0.30189 0.57837"
-        rpy="0 0 0" />
-      <mass
-        value="1.6794" />
-      <inertia
-        ixx="0.0079838"
-        ixy="8.7189E-06"
-        ixz="-4.4353E-05"
-        iyy="0.015974"
-        iyz="-2.3556E-06"
-        izz="0.022945" />
+        xyz="0.25112 -0.57291 0.30187"
+        rpy="0 0 0" />
+      <mass
+        value="1.633" />
+      <inertia
+        ixx="0.0079465"
+        ixy="4.4353E-05"
+        ixz="8.7912E-06"
+        iyy="0.022836"
+        iyz="2.3556E-06"
+        izz="0.015937" />
     </inertial>
     <visual>
@@ -28,5 +32,5 @@
         name="">
         <color
-          rgba="1 0.082353 0 1" />
+          rgba="0.79216 0.81961 0.93333 1" />
       </material>
     </visual>
@@ -42,291 +46,267 @@
   </link>
   <link
-    name="wheel1">
-    <inertial>
-      <origin
-        xyz="-0.0177039263600328 0.00801981738361954 -0.0194357011560703"
-        rpy="0 0 0" />
-      <mass
-        value="0.313742674369714" />
-      <inertia
-        ixx="0.000100019282088185"
-        ixy="-3.9651023978688E-06"
-        ixz="9.60926434754045E-06"
-        iyy="9.30624074713768E-05"
-        iyz="-4.35296350035507E-06"
-        izz="0.000101815459754744" />
-    </inertial>
-    <visual>
-      <origin
-        xyz="0 0 0"
-        rpy="0 0 0" />
-      <geometry>
-        <mesh
-          filename="file:///home/naveengnanasekar/dev_ws/src/my_robot/meshes/wheel1.STL" />
-      </geometry>
-      <material
-        name="">
-        <color
-          rgba="0.298039215686275 0.298039215686275 0.298039215686275 1" />
-      </material>
-    </visual>
-    <collision>
-      <origin
-        xyz="0 0 0"
-        rpy="0 0 0" />
-      <geometry>
-        <mesh
-          filename="file:///home/naveengnanasekar/dev_ws/src/my_robot/meshes/wheel1.STL" />
-      </geometry>
-    </collision>
-  </link>
-  <joint
-    name="w_joint_1"
-    type="revolute">
-    <origin
-      xyz="0.052037 -0.41904 0.45638"
-      rpy="2.7502 0.69985 -1.5135" />
-    <parent
-      link="base_link" />
-    <child
-      link="wheel1" />
-    <axis
-      xyz="0.6441 -0.29178 0.70711" />
-    <limit
-      lower="0"
-      upper="0"
-      effort="0"
-      velocity="0" />
-  </joint>
-  <link
-    name="wheel2">
-    <inertial>
-      <origin
-        xyz="1.38777878078145E-17 -3.33066907387547E-16 0.0274861360562049"
-        rpy="0 0 0" />
-      <mass
-        value="0.313742674369714" />
-      <inertia
-        ixx="9.12662298048282E-05"
-        ixy="-3.29019360449092E-19"
-        ixz="-2.13748764239623E-18"
-        iyy="9.12662298048309E-05"
-        iyz="5.65672424978063E-19"
-        izz="0.000112364689704675" />
-    </inertial>
-    <visual>
-      <origin
-        xyz="0 0 0"
-        rpy="0 0 0" />
-      <geometry>
-        <mesh
-          filename="file:///home/naveengnanasekar/dev_ws/src/my_robot/meshes/wheel2.STL" />
-      </geometry>
-      <material
-        name="">
-        <color
-          rgba="0.752941176470588 0.752941176470588 0.752941176470588 1" />
-      </material>
-    </visual>
-    <collision>
-      <origin
-        xyz="0 0 0"
-        rpy="0 0 0" />
-      <geometry>
-        <mesh
-          filename="file:///home/naveengnanasekar/dev_ws/src/my_robot/meshes/wheel2.STL" />
-      </geometry>
-    </collision>
-  </link>
-  <joint
-    name="w_joint_2"
-    type="revolute">
-    <origin
-      xyz="0.052037 -0.41904 0.091485"
-      rpy="0 0 0" />
-    <parent
-      link="base_link" />
-    <child
-      link="wheel2" />
+    name="W1">
+    <inertial>
+      <origin
+        xyz="-6.66133814775094E-16 7.21644966006352E-16 -0.0252070209755648"
+        rpy="0 0 0" />
+      <mass
+        value="0.219478804012584" />
+      <inertia
+        ixx="0.000194267977141188"
+        ixy="1.62630325872826E-19"
+        ixz="-1.3179284510751E-19"
+        iyy="0.000194267977141188"
+        iyz="-3.78873931579195E-21"
+        izz="0.000321855143610039" />
+    </inertial>
+    <visual>
+      <origin
+        xyz="0 0 0"
+        rpy="0 0 0" />
+      <geometry>
+        <mesh
+          filename="file:///home/naveengnanasekar/dev_ws/src/my_robot/meshes/W1.STL" />
+      </geometry>
+      <material
+        name="">
+        <color
+          rgba="0.792156862745098 0.819607843137255 0.933333333333333 1" />
+      </material>
+    </visual>
+    <collision>
+      <origin
+        xyz="0 0 0"
+        rpy="0 0 0" />
+      <geometry>
+        <mesh
+          filename="file:///home/naveengnanasekar/dev_ws/src/my_robot/meshes/W1.STL" />
+      </geometry>
+    </collision>
+  </link>
+  <joint
+    name="JOINT_WHEEL_1"
+    type="continuous">
+    <origin
+      xyz="0.052037 -0.41904 0.088366"
+      rpy="3.1416 0 -0.81731" />
+    <parent
+      link="base_link" />
+    <child
+      link="W1" />
+    <axis
+      xyz="0 0 1" />
+  </joint>
+  <link
+    name="W2">
+    <inertial>
+      <origin
+        xyz="1.66533453693773E-16 1.11022302462516E-16 0.0247929790244354"
+        rpy="0 0 0" />
+      <mass
+        value="0.219478804012584" />
+      <inertia
+        ixx="0.000194267977141189"
+        ixy="2.03287907341032E-19"
+        ixz="-6.07771461366044E-20"
+        iyy="0.000194267977141189"
+        iyz="-6.00962376213491E-20"
+        izz="0.00032185514361004" />
+    </inertial>
+    <visual>
+      <origin
+        xyz="0 0 0"
+        rpy="0 0 0" />
+      <geometry>
+        <mesh
+          filename="file:///home/naveengnanasekar/dev_ws/src/my_robot/meshes/W2.STL" />
+      </geometry>
+      <material
+        name="">
+        <color
+          rgba="0.792156862745098 0.819607843137255 0.933333333333333 1" />
+      </material>
+    </visual>
+    <collision>
+      <origin
+        xyz="0 0 0"
+        rpy="0 0 0" />
+      <geometry>
+        <mesh
+          filename="file:///home/naveengnanasekar/dev_ws/src/my_robot/meshes/W2.STL" />
+      </geometry>
+    </collision>
+  </link>
+  <joint
+    name="JOINT_WHEEL_2"
+    type="continuous">
+    <origin
+      xyz="0.052037 -0.41904 0.46447"
+      rpy="0 0 -0.30077" />
+    <parent
+      link="base_link" />
+    <child
+      link="W2" />
     <axis
       xyz="0 0 -1" />
-    <limit
-      lower="0"
-      upper="0"
-      effort="0"
-      velocity="0" />
-  </joint>
-  <link
-    name="wheel3">
-    <inertial>
-      <origin
-        xyz="-2.77555756156289E-16 -1.66533453693773E-16 -0.0274862321691448"
-        rpy="0 0 0" />
-      <mass
-        value="0.313742674369715" />
-      <inertia
-        ixx="9.12662298048202E-05"
-        ixy="-1.56833444140054E-19"
-        ixz="-2.83332520856563E-19"
-        iyy="9.12662298048205E-05"
-        iyz="5.91506929869319E-19"
-        izz="0.000112364689704665" />
-    </inertial>
-    <visual>
-      <origin
-        xyz="0 0 0"
-        rpy="0 0 0" />
-      <geometry>
-        <mesh
-          filename="file:///home/naveengnanasekar/dev_ws/src/my_robot/meshes/wheel3.STL" />
-      </geometry>
-      <material
-        name="">
-        <color
-          rgba="0.752941176470588 0.752941176470588 0.752941176470588 1" />
-      </material>
-    </visual>
-    <collision>
-      <origin
-        xyz="0 0 0"
-        rpy="0 0 0" />
-      <geometry>
-        <mesh
-          filename="file:///home/naveengnanasekar/dev_ws/src/my_robot/meshes/wheel3.STL" />
-      </geometry>
-    </collision>
-  </link>
-  <joint
-    name="w_joint_3"
-    type="revolute">
-    <origin
-      xyz="0.44204 -0.41904 0.45638"
-      rpy="3.1416 0 0" />
-    <parent
-      link="base_link" />
-    <child
-      link="wheel3" />
+  </joint>
+  <link
+    name="W3">
+    <inertial>
+      <origin
+        xyz="8.04911692853238E-15 -5.55111512312578E-15 -0.0252070209755648"
+        rpy="0 0 0" />
+      <mass
+        value="0.219478804012584" />
+      <inertia
+        ixx="0.000194267977141188"
+        ixy="2.60886147754325E-19"
+        ixz="3.45748612615907E-20"
+        iyy="0.000194267977141188"
+        iyz="2.48903131783379E-20"
+        izz="0.000321855143610039" />
+    </inertial>
+    <visual>
+      <origin
+        xyz="0 0 0"
+        rpy="0 0 0" />
+      <geometry>
+        <mesh
+          filename="file:///home/naveengnanasekar/dev_ws/src/my_robot/meshes/W3.STL" />
+      </geometry>
+      <material
+        name="">
+        <color
+          rgba="0.792156862745098 0.819607843137255 0.933333333333333 1" />
+      </material>
+    </visual>
+    <collision>
+      <origin
+        xyz="0 0 0"
+        rpy="0 0 0" />
+      <geometry>
+        <mesh
+          filename="file:///home/naveengnanasekar/dev_ws/src/my_robot/meshes/W3.STL" />
+      </geometry>
+    </collision>
+  </link>
+  <joint
+    name="JOINT_WHEEL_3"
+    type="continuous">
+    <origin
+      xyz="0.44204 -0.41904 0.088366"
+      rpy="-3.1416 0 0.21133" />
+    <parent
+      link="base_link" />
+    <child
+      link="W3" />
+    <axis
+      xyz="0 0 1" />
+  </joint>
+  <link
+    name="W4">
+    <inertial>
+      <origin
+        xyz="-3.77475828372553E-15 -1.11022302462516E-16 0.0247929790244354"
+        rpy="0 0 0" />
+      <mass
+        value="0.219478804012583" />
+      <inertia
+        ixx="0.000194267977141188"
+        ixy="2.16840434497101E-19"
+        ixz="-7.34324717805692E-20"
+        iyy="0.000194267977141188"
+        iyz="3.68119439514205E-19"
+        izz="0.000321855143610039" />
+    </inertial>
+    <visual>
+      <origin
+        xyz="0 0 0"
+        rpy="0 0 0" />
+      <geometry>
+        <mesh
+          filename="file:///home/naveengnanasekar/dev_ws/src/my_robot/meshes/W4.STL" />
+      </geometry>
+      <material
+        name="">
+        <color
+          rgba="0.792156862745098 0.819607843137255 0.933333333333333 1" />
+      </material>
+    </visual>
+    <collision>
+      <origin
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